File: pcb/v3/switching_circuit_v3/switching_circuit_v3.kicad_sch (KiCad schematic)
At the start: 128 parts, among them J2a Cell+, J2b Cell-, J3 OLED, J4 microSD, Q1 AO3400A, Q2 AO3400A, Q3 AO3400A, Q4 AO3400A, U1 UCC5304DWVR, U2 UCC5304DWVR, U3 UCC5304DWVR, U4 UCC5304DWVR

Commit message: V3: add placement guide, update KiCad layout and schematic
Add pcb/v3/PLACEMENT_GUIDE.md with checkboxed component placement map
organized by functional block (protection, power stage, gate drivers,
analog front-end, MCU, peripherals) for KiCad layout reference.

Co-Authored-By: Claude Opus 4.6 (1M context) <noreply@anthropic.com>
Parts:
- renumbered C_BTN_A to C_BTN_A1, C_BTN_B to C_BTN_B1, C_BTN_C to C_BTN_C1, D_LED_AUTO to D_LED_AUTO1, D_LED_PWR to D_LED_PWR1, D_LED_REC to D_LED_REC1, D_NEO to D_NEO1, D_TVS to D_TVS1, J2a to J2a1, J2b to J2b1, L_AVDD to L_AVDD1, Q_RP to Q_RP1, R_BTN_A to R_BTN_A1, R_BTN_B to R_BTN_B1, R_BTN_C to R_BTN_C1, R_CYC_GND to R_CYC_GND1, R_LED_AUTO to R_LED_AUTO1, R_LED_PWR to R_LED_PWR1, R_LED_REC to R_LED_REC1, R_RP to R_RP1, R_SCL to R_SCL1, R_SDA to R_SDA1, SW_A to SW_A1, SW_B to SW_B1, SW_C to SW_C1, TP_CYC_N to TP_CYC_N1, TP_CYC_P to TP_CYC_P1, TP_NEO_DIN to TP_NEO_DIN1, TP_NEO_GND to TP_NEO_GND1, TP_NEO_VDD to TP_NEO_VDD1
Other:
- moved on the sheet: C_BULK1, C_BULK2, D_TVS1, F1, Q1, Q_RP1, R_CYC_GND1, R_RP1, R_SH_P1, Rgpd_1, TP_CYC_N1, TP_CYC_P1
